File: pcb/v1/lul.brd (EAGLE design)
At the start: 90 x 96 mm, 86 parts, among them IC1 STM32F072C8T6, IC2 REG1117, IC3 74AHCT1G08DBV, U1 UG-2864HSWEG01

Commit message: working on v2
Parts:
- removed C26: 47uF, clock:C1210
- removed R1, R9: 5.1K, joyAnalog:0805
- removed U$8: USBC_16P, my_usbc_16p:USBC_16P_FOOT
- added R6: 300, clock:0805
- added S16, S17: ENCODER-SWITCH, SparkFun-Switches:ROTARY_ENC_PLAIN
- added X1: USB-MICROB, clock:USB-MICROB
- moved JP1 26.0 mm to (64.0, 76.0), turned to 0 degrees
- moved IC2 14.2 mm to (63.1, 85.0), turned to 90 degrees
- moved C27 13.6 mm to (69.3, 83.7), turned to 270 degrees
- moved U$10 10.8 mm to (71.0, 93.0)
- moved R5 6.30 mm to (55.9, 81.0)
- moved SD1 3.78 mm to (82.0, 67.0)
- moved IC3 2.58 mm to (57.0, 89.0)
- moved C9 0.06 mm to (69.5, 70.0)
Connections:
- removed net DNDNDN: IC1.32, U$8.A7, U$8.B7
- removed net N$31: R1.1, U$8.B5
- removed net N$33: R9.1, U$8.A5
- new net E1A: IC1.20, S17.A
- new net E1B: IC1.21, S17.B
- new net E1_SW: IC1.19, S17.SW+
- new net E2A: IC1.10, S16.A
- new net E2B: IC1.11, S16.B
- new net E2_SW: IC1.13, S16.SW-
- new net N$16: IC1.17, R6.1
- new net USB_DN: IC1.32, X1.D-
- net GND: now also S16.C, S16.SW+, S17.C, S17.SW-, X1.GND, X1.P1, X1.P2, X1.P3, X1.P4, X1.P5, X1.P6; no longer C26.2, R1.2, R9.2, U$8.A1B12, U$8.B11A12, U$8.P$13, U$8.P$14, U$8.P$15, U$8.P$16
- net N$1: now also X1.VBUS; no longer C26.1, U$8.A4B9, U$8.B4A9
- net SPI_MOSI: now also R6.2; no longer IC1.17
- net USB_DP: now also X1.D+; no longer U$8.A6, U$8.B6
Routing:
- net N$32: track 54.7 -> 8.26 mm
- net N$34: track 50.5 -> 5.83 mm
- net UART1_TX: track 38.4 -> 5.93 mm
- net E1_SW: track 0.00 -> 27.9 mm
- net E1A: track 0.00 -> 25.6 mm
- net E2_SW: track 0.00 -> 24.7 mm
- net DNDNDN: track 23.3 -> 0.00 mm
- net SW3: track 20.9 -> 44.0 mm
- net USB_DN: track 0.00 -> 22.2 mm
- net E2B: track 0.00 -> 20.3 mm
- net GND: track 48.6 -> 28.5 mm
- net E1B: track 0.00 -> 18.7 mm
- net SW2: track 46.4 -> 63.5 mm
- net SW1: track 67.5 -> 83.3 mm
- net E2A: track 0.00 -> 13.8 mm
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