File: pcb/v1/lul.sch (EAGLE design)
At the start: 86 parts, among them IC1 STM32F072C8T6, IC2 REG1117, IC3 74AHCT1G08DBV, U1 UG-2864HSWEG01

Commit message: working on v2
Parts:
- removed C26: 47uF, clock:C-USC1210
- removed R1, R9: 5.1K, joyAnalog:RESISTOR0805-RES
- removed U$8: USBC_16P, my_usbc_16p:USBC_16P
- added R6: 300, clock:RESISTOR0805-RES
- added S16, S17: ENCODER-SWITCH, SparkFun-Switches:ENCODER-SWITCH
- added X1: USB-MICROB, clock:USB-MICROB
Connections:
- removed net DNDNDN: IC1PORTA_H.PA11, U$8.DN1, U$8.DN2
- removed net N$31: R1.1, U$8.CC2
- removed net N$33: R9.1, U$8.CC1
- new net E1A: IC1PORTB_L.PB2, S17.A
- new net E1B: IC1PORTB_H.PB10, S17.B
- new net E1_SW: IC1PORTB_L.PB1, S17.SW+
- new net E2A: IC1PORTA_L.PA0, S16.A
- new net E2B: IC1PORTA_L.PA1, S16.B
- new net E2_SW: IC1PORTA_L.PA3, S16.SW-
- new net N$16: IC1PORTA_L.PA7, R6.1
- new net USB_DN: IC1PORTA_H.PA11, X1.D-
- net GND: now also S16.C, S16.SW+, S17.C, S17.SW-, X1.GND; no longer C26.2, R1.2, R9.2, U$8.GND
- net N$1: now also X1.VBUS; no longer C26.1, U$8.VBUS
- net SPI_MOSI: now also R6.2; no longer IC1PORTA_L.PA7
- net USB_DP: now also X1.D+; no longer U$8.DP1, U$8.DP2
