File: pcb/V2/lul.sch (EAGLE design)
At the start: 85 parts, among them IC1 STM32F072C8T6, IC2 REG1117, IC3 74AHCT1G08DBV, SW1 324_SW324_SWITCH_FOOT_HOLE, SW10 KAILH_SWITCH_SOCKET, SW11 KAILH_SWITCH_SOCKET, SW12 KAILH_SWITCH_SOCKET, SW13 KAILH_SWITCH_SOCKET, SW14 KAILH_SWITCH_SOCKET, SW15 KAILH_SWITCH_SOCKET, SW16 KAILH_SWITCH_SOCKET, SW17 KAILH_SWITCH_SOCKET, SW18 KAILH_SWITCH_SOCKET, SW19 KAILH_SWITCH_SOCKET, SW2 324_SW324_SWITCH_FOOT_HOLE, SW3 324_SW324_SWITCH_FOOT_HOLE, SW4 324_SW324_SWITCH_FOOT_HOLE, SW5 KAILH_SWITCH_SOCKET, SW6 KAILH_SWITCH_SOCKET, SW7 KAILH_SWITCH_SOCKET, SW8 KAILH_SWITCH_SOCKET, SW9 KAILH_SWITCH_SOCKET, U1 UG-2864HSWEG01, U2 USBC_16P

Commit message: added hot-swap sockets
Parts:
- removed SW10, SW11, SW12, SW13, SW14, SW15, SW16, SW17, SW18, SW19, SW5, SW6, SW7, SW8, SW9: KAILH_SWITCH_SOCKET, Kailh_switch_socket:KAILH_SWITCH_SOCKET
- added S1, S10, S11, S12, S13, S14, S15, S2, S3, S4, S5, S6, S7, S8, S9: CHERRY-MX-LED, SparkFun-Cherry-MX-Switch-Breakout:CHERRY-MX-LED
Connections:
- net GND: now also S1.S2, S10.S2, S11.S2, S12.S2, S13.S2, S14.S2, S15.S2, S2.S2, S3.S2, S4.S2, S5.S2, S6.S2, S7.S2, S8.S2, S9.S2; no longer SW10.2, SW11.2, SW12.2, SW13.2, SW14.2, SW15.2, SW16.2, SW17.2, SW18.2, SW19.2, SW5.2, SW6.2, SW7.2, SW8.2, SW9.2
- net SW1: now also S1.S1; no longer SW5.1
- net SW10: now also S10.S1; no longer SW14.1
- net SW11: now also S11.S1; no longer SW15.1
- net SW12: now also S12.S1; no longer SW16.1
- net SW13: now also S13.S1; no longer SW17.1
- net SW14: now also S14.S1; no longer SW18.1
- net SW15: now also S15.S1; no longer SW19.1
- net SW2: now also S2.S1; no longer SW6.1
- net SW3: now also S3.S1; no longer SW7.1
- net SW4: now also S4.S1; no longer SW8.1
- net SW5: now also S5.S1; no longer SW9.1
- net SW6: now also S6.S1; no longer SW10.1
- net SW7: now also S7.S1; no longer SW11.1
- net SW8: now also S8.S1; no longer SW12.1
- net SW9: now also S9.S1; no longer SW13.1
