File: pcb/V3/lul.brd (EAGLE design)
At the start: 90 x 96 mm, 85 parts, among them IC1 STM32F072C8T6, IC2 REG1117, IC3 74AHCT1G08DBV, SW1 324_SW324_SWITCH_FOOT_HOLE, SW10 KAILH_SWITCH_SOCKET, SW11 KAILH_SWITCH_SOCKET, SW12 KAILH_SWITCH_SOCKET, SW13 KAILH_SWITCH_SOCKET, SW14 KAILH_SWITCH_SOCKET, SW15 KAILH_SWITCH_SOCKET, SW16 KAILH_SWITCH_SOCKET, SW17 KAILH_SWITCH_SOCKET, SW18 KAILH_SWITCH_SOCKET, SW19 KAILH_SWITCH_SOCKET, SW2 324_SW324_SWITCH_FOOT_HOLE, SW3 324_SW324_SWITCH_FOOT_HOLE, SW4 324_SW324_SWITCH_FOOT_HOLE, SW5 KAILH_SWITCH_SOCKET, SW6 KAILH_SWITCH_SOCKET, SW7 KAILH_SWITCH_SOCKET, SW8 KAILH_SWITCH_SOCKET, SW9 KAILH_SWITCH_SOCKET, U1 UG-2864HSWEG01, U2 USBC_16P

Commit message: changed to reverse-mount RGB LED
Parts:
- LED1, LED10, LED11, LED12, LED13, LED14, LED15, LED2, LED3, LED4, LED5, LED6, LED7, LED8, LED9: value WS2812B -> WS2812B3535; device lul:REVERSE_MNT -> lul:LED3535
- moved C21 7.11 mm to (48.0, 75.0), flipped to the top, turned to 180 degrees
- moved C11 6.99 mm to (29.0, 37.0), flipped to the top, turned to 180 degrees
- moved C19 6.98 mm to (10.0, 75.0), flipped to the top, turned to 180 degrees
- moved R5 6.93 mm to (56.7, 87.3), flipped to the top, turned to 90 degrees
- moved C20 6.92 mm to (29.0, 75.0), flipped to the top, turned to 180 degrees
- moved C25 6.91 mm to (10.0, 37.0), flipped to the top, turned to 180 degrees
- moved C12 6.86 mm to (48.0, 37.0), flipped to the top, turned to 180 degrees
- moved C18 6.59 mm to (48.0, 94.0), flipped to the top, turned to 0 degrees
- moved C23 6.59 mm to (29.0, 56.0), flipped to the top, turned to 0 degrees
- moved C14 6.58 mm to (29.0, 18.0), flipped to the top, turned to 0 degrees
- moved C17 6.57 mm to (29.0, 94.0), flipped to the top, turned to 0 degrees
- moved C22 6.57 mm to (10.0, 56.0), flipped to the top, turned to 0 degrees
- moved C15 6.48 mm to (48.0, 18.0), flipped to the top, turned to 0 degrees
- moved C24 6.46 mm to (48.0, 56.0), flipped to the top, turned to 0 degrees
- moved IC3 5.09 mm to (59.6, 89.5), flipped to the top, turned to 0 degrees
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Connections:
- net +3V3: now also LED1.2, LED10.2, LED11.2, LED12.2, LED13.2, LED14.2, LED15.2, LED2.2, LED3.2, LED4.2, LED5.2, LED6.2, LED7.2, LED8.2, LED9.2; no longer LED1.VDD, LED10.VDD, LED11.VDD, LED12.VDD, LED13.VDD, LED14.VDD, LED15.VDD, LED2.VDD, LED3.VDD, LED4.VDD, LED5.VDD, LED6.VDD, LED7.VDD, LED8.VDD, LED9.VDD
- net GND: now also LED1.4, LED10.4, LED11.4, LED12.4, LED13.4, LED14.4, LED15.4, LED2.4, LED3.4, LED4.4, LED5.4, LED6.4, LED7.4, LED8.4, LED9.4; no longer LED1.GND, LED10.GND, LED11.GND, LED12.GND, LED13.GND, LED14.GND, LED15.GND, LED2.GND, LED3.GND, LED4.GND, LED5.GND, LED6.GND, LED7.GND, LED8.GND, LED9.GND
- net N$15: now also LED1.1, LED2.3; no longer LED1.DIN, LED2.DOUT
- net N$17: now also LED1.3, LED4.1; no longer LED1.DOUT, LED4.DIN
- net N$18: now also LED4.3, LED5.1; no longer LED4.DOUT, LED5.DIN
- net N$19: now also LED5.3, LED6.1; no longer LED5.DOUT, LED6.DIN
- net N$20: now also LED6.3, LED9.1; no longer LED6.DOUT, LED9.DIN
- net N$21: now also LED8.1, LED9.3; no longer LED8.DIN, LED9.DOUT
- net N$22: now also LED7.1, LED8.3; no longer LED7.DIN, LED8.DOUT
- net N$23: now also LED10.1, LED7.3; no longer LED10.DIN, LED7.DOUT
- net N$24: now also LED10.3, LED11.1; no longer LED10.DOUT, LED11.DIN
- net N$25: now also LED11.3, LED12.1; no longer LED11.DOUT, LED12.DIN
- net N$26: now also LED12.3, LED15.1; no longer LED12.DOUT, LED15.DIN
- net N$27: now also LED14.1, LED15.3; no longer LED14.DIN, LED15.DOUT
- net N$28: now also LED13.1, LED14.3; no longer LED13.DIN, LED14.DOUT
- net N$29: now also LED3.1; no longer LED3.DIN
- net N$9: now also LED2.1, LED3.3; no longer LED2.DIN, LED3.DOUT
Routing:
- net GND: track 228.7 -> 172.6 mm, vias 49 -> 18
- net +3V3: track 109.4 -> 127.3 mm, vias 10 -> 26
- net LED_DATA_EN: track 36.8 -> 21.7 mm, vias 1 -> 2
- net N$29: track 3.75 -> 12.0 mm
- net SPI_MOSI: track 42.1 -> 35.7 mm, vias 1 -> 2
- net N$23: track 27.8 -> 25.7 mm
- net SW14: track 74.2 -> 72.2 mm
- net SW13: track 92.5 -> 90.6 mm
- net SW1: track 65.2 -> 67.1 mm
- net SW4: track 52.6 -> 54.4 mm, vias 3 -> 1
- net SW2: track 44.5 -> 46.2 mm
- net N$9: track 14.6 -> 16.2 mm
- net N$28: track 14.6 -> 16.2 mm
- net N$27: track 14.6 -> 16.2 mm
- net N$25: track 14.6 -> 16.2 mm
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Other:
- board text added: "dekuNukem PD2 MAY20"
- board text removed: "dekuNukem PT4 MAY2020"
