File: pcb/V3/lul.sch (EAGLE design)
At the start: 85 parts, among them IC1 STM32F072C8T6, IC2 REG1117, IC3 74AHCT1G08DBV, SW1 324_SW324_SWITCH_FOOT_HOLE, SW10 KAILH_SWITCH_SOCKET, SW11 KAILH_SWITCH_SOCKET, SW12 KAILH_SWITCH_SOCKET, SW13 KAILH_SWITCH_SOCKET, SW14 KAILH_SWITCH_SOCKET, SW15 KAILH_SWITCH_SOCKET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

Commit message: changed to reverse-mount RGB LED
Parts:
- LED1, LED10, LED11, LED12, LED13, LED14, LED15, LED2, LED3, LED4, LED5, LED6, LED7, LED8, LED9: value WS2812B -> WS2812B3535; device lul:WS2812B -> lul:WS2812B3535
Changed lines of the file:
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@@
 <part name="GND45" library="backplane" deviceset="GND" device=""/>
 <part name="GND19" library="supply1" library_urn="urn:adsk.eagle:library:371" deviceset="GND" device=""/>
-<part name="LED1" library="lul" deviceset="WS2812B" device="" value="WS2812B"/>
+<part name="LED1" library="lul" deviceset="WS2812B" device="3535"/>
 <part name="GND1" library="supply1" library_urn="urn:adsk.eagle:library:371" deviceset="GND" device=""/>
-<part name="LED2" library="lul" deviceset="WS2812B" device="" value="WS2812B"/>
-<part name="LED3" library="lul" deviceset="WS2812B" device="" value="WS2812B"/>
-<part name="LED4" library="lul" deviceset="WS2812B" device="" value="WS2812B"/>
-<part name="LED5" library="lul" deviceset="WS2812B" device="" value="WS2812B"/>
-<part name="LED6" library="lul" deviceset="WS2812B" device="" value="WS2812B"/>
-<part name="LED7" library="lul" deviceset="WS2812B" device="" value="WS2812B"/>
-<part name="LED8" library="lul" deviceset="WS2812B" device="" value="WS2812B"/>
-<part name="LED9" library="lul" deviceset="WS2812B" device="" value="WS2812B"/>
-<part name="LED10" library="lul" deviceset="WS2812B" device="" value="WS2812B"/>
-<part name="LED11" library="lul" deviceset="WS2812B" device="" value="WS2812B"/>
-<part name="LED12" library="lul" deviceset="WS2812B" device="" value="WS2812B"/>
-<part name="LED13" library="lul" deviceset="WS2812B" device="" value="WS2812B"/>
-<part name="LED14" library="lul" deviceset="WS2812B" device="" value="WS2812B"/>
-<part name="LED15" library="lul" deviceset="WS2812B" device="" value="WS2812B"/>
+<part name="LED2" library="lul" deviceset="WS2812B" device="3535"/>
+<part name="LED3" library="lul" deviceset="WS2812B" device="3535"/>
+<part name="LED4" library="lul" deviceset="WS2812B" device="3535"/>
+<part name="LED5" library="lul" deviceset="WS2812B" device="3535"/>
+<part name="LED6" library="lul" deviceset="WS2812B" device="3535"/>
+<part name="LED7" library="lul" deviceset="WS2812B" device="3535"/>
+<part name="LED8" library="lul" deviceset="WS2812B" device="3535"/>
+<part name="LED9" library="lul" deviceset="WS2812B" device="3535"/>
+<part name="LED10" library="lul" deviceset="WS2812B" device="3535"/>
+<part name="LED11" library="lul" deviceset="WS2812B" device="3535"/>
+<part name="LED12" library="lul" deviceset="WS2812B" device="3535"/>
+<part name="LED13" library="lul" deviceset="WS2812B" device="3535"/>
+<part name="LED14" library="lul" deviceset="WS2812B" device="3535"/>
+<part name="LED15" library="lul" deviceset="WS2812B" device="3535"/>
 <part name="+3V11" library="supply1" library_urn="urn:adsk.eagle:library:371" deviceset="+3V3" device=""/>
 <part name="+3V12" library="supply1" library_urn="urn:adsk.eagle:library:371" deviceset="+3V3" device=""/>
