File: pcb/V4/lul.brd (EAGLE design)
At the start: 90 x 96 mm, 90 parts, among them IC1 STM32F072C8T6, IC2 REG1117, IC3 74AHCT1G08DBV, SW1 324_SW324_SWITCH_FOOT_HOLE, SW10 KAILH_SWITCH_SOCKET, SW11 KAILH_SWITCH_SOCKET, SW12 KAILH_SWITCH_SOCKET, SW13 KAILH_SWITCH_SOCKET, SW14 KAILH_SWITCH_SOCKET, SW15 KAILH_SWITCH_SOCKET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

Commit message: modified mounting plate design
Parts:
- removed U$12, U$13, U$17, U$22, U$23, U$8: M2_SCREW_DEV, 3pos_slide_switch_centered:M2_SCREW_FOOT
- added U$14: M3_MOUNTING_HOLE, clock:M3_MOUNTING_HOLE_PACK
- U$10, U$11, U$15, U$16, U$7, U$9: value M2_SCREW_DEV -> M3_MOUNTING_HOLE; device 3pos_slide_switch_centered:M2_SCREW_FOOT -> clock:M3_MOUNTING_HOLE_PACK
- moved U$9 51.6 mm to (86.5, 57.5)
- moved SW1 27.6 mm to (60.7, 51.6), turned to 270 degrees
- moved R2 24.9 mm to (60.7, 55.5), turned to 0 degrees
- moved SW2 23.2 mm to (65.8, 51.6)
- moved R4 19.8 mm to (65.8, 55.5), turned to 0 degrees
- moved C28 2.00 mm to (76.8, 49.8)
- moved C3 2.00 mm to (69.1, 48.1)
- moved C4 2.00 mm to (72.2, 48.1)
- moved C5 2.00 mm to (81.0, 49.8)
- moved C6 2.00 mm to (69.1, 50.2)
- moved C7 2.00 mm to (69.1, 51.7)
- moved C8 2.00 mm to (78.7, 48.1)
- moved R3 2.00 mm to (75.7, 48.1)
- moved R7 2.00 mm to (69.1, 53.6)
- moved R8 2.00 mm to (69.1, 55.5)
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Routing:
- net GND: track 183.8 -> 228.7 mm
- net N$2: track 38.7 -> 18.2 mm
- net RST: track 30.5 -> 13.0 mm
- net SCL: track 29.6 -> 33.2 mm
- net SDA: track 34.4 -> 37.3 mm
- net N$34: track 52.9 -> 50.5 mm
- net BUTTON1: track 74.6 -> 72.8 mm
- net BUTTON2: track 87.9 -> 86.4 mm
- net OLED_RESET: track 16.8 -> 18.2 mm
- net +3V3: track 108.5 -> 109.4 mm, vias 11 -> 10
- net LED_DATA_EN: track 37.3 -> 36.8 mm
