File: pcb/V6/lul.sch (EAGLE design)
At the start: 90 parts, among them IC1 STM32F072C8T6, IC2 REG1117, IC3 74AHCT1G08DBV, SW1 324_SW324_SWITCH_FOOT_HOLE, SW10 KAILH_SWITCH_SOCKET, SW11 KAILH_SWITCH_SOCKET, SW12 KAILH_SWITCH_SOCKET, SW13 KAILH_SWITCH_SOCKET, SW14 KAILH_SWITCH_SOCKET, SW15 KAILH_SWITCH_SOCKET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

Commit message: getting ready for a new production run
Parts:
- R17, R2, R4, R5: value 5.1K -> 10K
Changed lines of the file:
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@@
 <part name="GND7" library="supply1" library_urn="urn:adsk.eagle:library:371" deviceset="GND" device=""/>
 <part name="+3V5" library="supply1" library_urn="urn:adsk.eagle:library:371" deviceset="+3V3" device=""/>
-<part name="R2" library="clock" deviceset="RESISTOR" device="0805-RES" value="5.1K"/>
-<part name="R4" library="clock" deviceset="RESISTOR" device="0805-RES" value="5.1K"/>
+<part name="R2" library="clock" deviceset="RESISTOR" device="0805-RES" value="10K"/>
+<part name="R4" library="clock" deviceset="RESISTOR" device="0805-RES" value="10K"/>
 <part name="GND9" library="supply1" library_urn="urn:adsk.eagle:library:371" deviceset="GND" device=""/>
 <part name="+3V6" library="supply1" library_urn="urn:adsk.eagle:library:371" deviceset="+3V3" device=""/>
@@
 <part name="U$3" library="supply1" library_urn="urn:adsk.eagle:library:371" deviceset="GND" device=""/>
 <part name="+3V2" library="supply1" library_urn="urn:adsk.eagle:library:371" deviceset="+3V3" device=""/>
-<part name="R17" library="clock" deviceset="RESISTOR" device="0805-RES" value="5.1K"/>
+<part name="R17" library="clock" deviceset="RESISTOR" device="0805-RES" value="10K"/>
 <part name="GND45" library="backplane" deviceset="GND" device=""/>
 <part name="GND19" library="supply1" library_urn="urn:adsk.eagle:library:371" deviceset="GND" device=""/>
@@
 <part name="U$6" library="supply1" library_urn="urn:adsk.eagle:library:371" deviceset="GND" device=""/>
 <part name="+3V30" library="supply1" library_urn="urn:adsk.eagle:library:371" deviceset="+3V3" device=""/>
-<part name="R5" library="clock" deviceset="RESISTOR" device="0805-RES" value="5.1K"/>
+<part name="R5" library="clock" deviceset="RESISTOR" device="0805-RES" value="10K"/>
 <part name="GND32" library="supply1" library_urn="urn:adsk.eagle:library:371" deviceset="GND" device=""/>
 <part name="+3V32" library="supply1" library_urn="urn:adsk.eagle:library:371" deviceset="+3V3" device=""/>
