File: pcb/V3_PD1/lul.brd (EAGLE design)
At the start: 90 x 96 mm, 95 parts, among them IC1 STM32F072C8T6, IC2 REG1117, IC3 74AHCT1G08DBV, SW1 324_SW324_SWITCH_FOOT_HOLE, SW10 KAILH_SWITCH_SOCKET, SW11 KAILH_SWITCH_SOCKET, SW12 KAILH_SWITCH_SOCKET, SW13 KAILH_SWITCH_SOCKET, SW14 KAILH_SWITCH_SOCKET, SW15 KAILH_SWITCH_SOCKET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

Commit message: slightly updated pcb design for new production run
Parts:
- removed TP1, TP2, TP3, TP5: PTR1TP11SQ, testpad:TP11SQ
- removed TP4: PTR1TP09R, testpad:TP09R
- moved C16 0.05 mm to (8.35, 93.9)
Connections:
- removed net N$13: IC1.20, TP2.TP
- removed net N$16: IC1.21, TP3.TP
- removed net N$2: IC1.19, TP1.TP
- removed net N$30: IC1.22, TP4.TP
- removed net N$35: IC1.25, TP5.TP
Routing:
- net N$35: track 5.55 -> 0.00 mm, vias 1 -> 0
- net GND: track 225.7 -> 220.2 mm, vias 51 -> 49
- net N$2: track 4.28 -> 0.00 mm, vias 1 -> 0
- net N$13: track 3.40 -> 0.00 mm, vias 1 -> 0
- net N$16: track 3.03 -> 0.00 mm, vias 1 -> 0
- net SDA: track 38.1 -> 35.4 mm
- net N$30: track 1.53 -> 0.00 mm
- net +3V3: track 99.6 -> 101.0 mm
Other:
- board text added: "dekuNukem PD2 AUG2020"
- board text added: "duckypad"
- board text removed: "PB1"
- board text removed: "PB10"
- board text removed: "PB11"
- board text removed: "PB12"
- board text removed: "PB2"
- board text removed: "dekuNukem PD2 DEC2020"
- board text removed: "duckyPad V3"
