File: pcb/V3_PD1/lul.sch (EAGLE design)
At the start: 95 parts, among them IC1 STM32F072C8T6, IC2 REG1117, IC3 74AHCT1G08DBV, SW1 324_SW324_SWITCH_FOOT_HOLE, SW10 KAILH_SWITCH_SOCKET, SW11 KAILH_SWITCH_SOCKET, SW12 KAILH_SWITCH_SOCKET, SW13 KAILH_SWITCH_SOCKET, SW14 KAILH_SWITCH_SOCKET, SW15 KAILH_SWITCH_SOCKET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

Commit message: slightly updated pcb design for new production run
Parts:
- removed TP1, TP2, TP3, TP5: PTR1TP11SQ, testpad:PTR1TP11SQ
- removed TP4: PTR1TP09R, testpad:PTR1TP09R
Connections:
- removed net N$13: IC1PORTB_L.PB2, TP2.TP
- removed net N$16: IC1PORTB_H.PB10, TP3.TP
- removed net N$2: IC1PORTB_L.PB1, TP1.TP
- removed net N$30: IC1PORTB_H.PB11, TP4.TP
- removed net N$35: IC1PORTB_H.PB12, TP5.TP
Changed lines of the file:
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@@
 <part name="U$23" library="3pos_slide_switch_centered" deviceset="M2_SCREW_DEV" device=""/>
 <part name="U$14" library="3pos_slide_switch_centered" deviceset="M2_SCREW_DEV" device=""/>
-<part name="TP1" library="testpad" library_urn="urn:adsk.eagle:library:385" deviceset="PTR1" device="TP11SQ" package3d_urn="urn:adsk.eagle:package:27965/1" value="PTR1TP11SQ"/>
-<part name="TP2" library="testpad" library_urn="urn:adsk.eagle:library:385" deviceset="PTR1" device="TP11SQ" package3d_urn="urn:adsk.eagle:package:27965/1" value="PTR1TP11SQ"/>
-<part name="TP3" library="testpad" library_urn="urn:adsk.eagle:library:385" deviceset="PTR1" device="TP11SQ" package3d_urn="urn:adsk.eagle:package:27965/1" value="PTR1TP11SQ"/>
-<part name="TP4" library="testpad" library_urn="urn:adsk.eagle:library:385" deviceset="PTR1" device="TP09R" package3d_urn="urn:adsk.eagle:package:27958/1" value="PTR1TP09R"/>
-<part name="TP5" library="testpad" library_urn="urn:adsk.eagle:library:385" deviceset="PTR1" device="TP11SQ" package3d_urn="urn:adsk.eagle:package:27965/1" value="PTR1TP11SQ"/>
 </parts>
 <sheets>
@@
 <instance part="U$23" gate="G$1" x="558.8" y="27.94" smashed="yes"/>
 <instance part="U$14" gate="G$1" x="520.7" y="-20.32" smashed="yes"/>
-<instance part="TP1" gate="G$1" x="464.82" y="-157.48" smashed="yes" rot="R90">
-<attribute name="NAME" x="471.17" y="-158.496" size="1.778" layer="95" rot="R180"/>
-<attribute name="TP_SIGNAL_NAME" x="467.36" y="-156.21" size="1.778" layer="97" rot="R90"/>
-</instance>
-<instance part="TP2" gate="G$1" x="482.6" y="-160.02" smashed="yes" rot="R90">
-<attribute name="NAME" x="488.95" y="-161.036" size="1.778" layer="95" rot="R180"/>
-<attribute name="TP_SIGNAL_NAME" x="485.14" y="-158.75" size="1.778" layer="97" rot="R90"/>
-</instance>
-<instance part="TP3" gate="G$1" x="457.2" y="-187.96" smashed="yes" rot="R90">
-<attribute name="NAME" x="463.55" y="-188.976" size="1.778" layer="95" rot="R180"/>
-<attribute name="TP_SIGNAL_NAME" x="459.74" y="-186.69" size="1.778" layer="97" rot="R90"/>
-</instance>
-<instance part="TP4" gate="G$1" x="469.9" y="-190.5" smashed="yes" rot="R90">
-<attribute name="NAME" x="476.25" y="-191.516" size="1.778" layer="95" rot="R180"/>
-<attribute name="TP_SIGNAL_NAME" x="472.44" y="-189.23" size="1.778" layer="97" rot="R90"/>
-</instance>
-<instance part="TP5" gate="G$1" x="482.6" y="-193.04" smashed="yes" rot="R90">
-<attribute name="NAME" x="488.95" y="-194.056" size="1.778" layer="95" rot="R180"/>
-<attribute name="TP_SIGNAL_NAME" x="485.14" y="-191.77" size="1.778" layer="97" rot="R90"/>
-</instance>
 </instances>
 <busses>
@@
 </segment>
 </net>
-<net name="N$2" class="0">
-<segment>
-<pinref part="IC1" gate="PORTB_L" pin="PB1"/>
-<pinref part="TP1" gate="G$1" pin="TP"/>
-<wire x1="434.34" y1="-157.48" x2="462.28" y2="-157.48" width="0.1524" layer="91"/>
-</segment>
-</net>
-<net name="N$13" class="0">
-<segment>
-<pinref part="IC1" gate="PORTB_L" pin="PB2"/>
-<pinref part="TP2" gate="G$1" pin="TP"/>
-<wire x1="434.34" y1="-160.02" x2="480.06" y2="-160.02" width="0.1524" layer="91"/>
-</segment>
-</net>
-<net name="N$16" class="0">
-<segment>
-<pinref part="IC1" gate="PORTB_H" pin="PB10"/>
-<pinref part="TP3" gate="G$1" pin="TP"/>
-<wire x1="434.34" y1="-187.96" x2="454.66" y2="-187.96" width="0.1524" layer="91"/>
-</segment>
-</net>
-<net name="N$30" class="0">
-<segment>
-<pinref part="IC1" gate="PORTB_H" pin="PB11"/>
-<pinref part="TP4" gate="G$1" pin="TP"/>
-<wire x1="434.34" y1="-190.5" x2="467.36" y2="-190.5" width="0.1524" layer="91"/>
-</segment>
-</net>
-<net name="N$35" class="0">
-<segment>
-<pinref part="IC1" gate="PORTB_H" pin="PB12"/>
-<pinref part="TP5" gate="G$1" pin="TP"/>
-<wire x1="434.34" y1="-193.04" x2="480.06" y2="-193.04" width="0.1524" layer="91"/>
-</segment>
-</net>
 </nets>
 </sheet>
@@
 with this version.
 </note>
-<note version="8.3" severity="warning">
-Since Version 8.3, EAGLE supports URNs for individual library
-assets (packages, symbols, and devices). The URNs of those assets
-will not be understood (or retained) with this version.
-</note>
-<note version="8.3" severity="warning">
-Since Version 8.3, EAGLE supports the association of 3D packages
-with devices in libraries, schematics, and board files. Those 3D
-packages will not be understood (or retained) with this version.
-</note>
 </compatibility>
