File: pcb/duckypad2020_v4.brd (EAGLE design)
At the start: 90 x 96 mm, 98 parts, among them IC1 STM32F072C8T6, IC2 REG1117, IC3 74AHCT1G08DBV, SW1 324_SW324_SWITCH_FOOT_HOLE, SW10 KAILH_SWITCH_SOCKET_KAILH_SWI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, SW11 KAILH_SWITCH_SOCKET_KAILH_SWI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, SW12 KAILH_SWITCH_SOCKET_KAILH_SWI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, SW13 KAILH_SWITCH_SOCKET_KAILH_SWI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, SW14 KAILH_SWITCH_SOCKET_KAILH_SWI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, SW15 KAILH_SWITCH_SOCKET_KAILH_SWI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

Commit message: clean up files
Parts:
- removed R10, R6: 5.1K, joyAnalog:0805
- removed SH1: SH10P, duckypad:DUCKYPAD_SM12B-SSR-H-TB
- removed U3: USBC_16P, my_usbc_16p:USBC_16P_FOOT
Connections:
- removed net +5V: C29.2, IC2.3, SH1.1, U2.A4B9, U2.B4A9, U3.A4B9, U3.B4A9
- removed net N$36: R6.1, U3.B5
- removed net N$37: R10.1, U3.A5
- new net N$1: C29.2, IC2.3, U2.A4B9, U2.B4A9
- net +3V3: no longer SH1.3
- net BUTTON_DEBUG: now also IC1.13
- net GND: no longer R10.2, R6.2, SH1.2, SH1.FIT@1, SH1.FIT@2, U3.A1B12, U3.B11A12, U3.P$13, U3.P$14, U3.P$15, U3.P$16
Routing:
- net N$1: track 0.00 -> 13.8 mm, vias 0 -> 2
- net +5V: track 13.8 -> 0.00 mm, vias 2 -> 0
- net BUTTON_DEBUG: track 41.1 -> 45.2 mm, vias 2 -> 3
Other:
- board text added: "duckyPad V4"
- board text removed: "duckyPad V3.1"

Commit message: adding components
Parts:
- added R10, R6: 5.1K, joyAnalog:0805
- added SH1: SH10P, duckypad:DUCKYPAD_SM12B-SSR-H-TB
- added U3: USBC_16P, my_usbc_16p:USBC_16P_FOOT
Connections:
- new net +5V: C29.2, IC2.3, SH1.1, U2.A4B9, U2.B4A9
- new net N$36: R10.1, U3.A5
- net +3V3: now also SH1.3
- net GND: now also R10.2, R6.2, SH1.2, SH1.FIT@1, SH1.FIT@2, U3.A1B12, U3.B11A12, U3.P$13, U3.P$14, U3.P$15, U3.P$16
- net N$1: now also R6.1, U3.B5; no longer C29.2, IC2.3, U2.A4B9, U2.B4A9
Routing:
- net N$1: track 13.8 -> 0.00 mm, vias 2 -> 0
- net +5V: track 0.00 -> 13.8 mm, vias 0 -> 2
Changed lines of the file:
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@@
 <element name="SW21" library="duckypad" package="EVQ-Q2" value="SPST_TACT-EVQQ2" x="65" y="7.5" smashed="yes"/>
 <element name="U$14" library="adafruit_changed" package="1X02" value="PINHD1X2" x="88.9" y="66.675" smashed="yes" rot="R270"/>
+<element name="SH1" library="duckypad" package="DUCKYPAD_SM12B-SSR-H-TB" value="SH10P" x="86.614" y="20.574" smashed="yes" rot="MR90"/>
+<element name="U3" library="my_usbc_16p" package="USBC_16P_FOOT" value="USBC_16P" x="85.852" y="33.401" smashed="yes" rot="MR90"/>
+<element name="R6" library="joyAnalog" package="0805" value="5.1K" x="63.5" y="33.274" smashed="yes" rot="MR0">
+<attribute name="NAME" x="64.262" y="34.0995" size="0.8128" layer="26" rot="MR0"/>
+</element>
+<element name="R10" library="joyAnalog" package="0805" value="5.1K" x="68.707" y="37.973" smashed="yes" rot="MR0">
+<attribute name="NAME" x="69.469" y="38.7985" size="0.8128" layer="26" rot="MR0"/>
+</element>
 </elements>
 <signals>
@@
 <wire x1="3.645" y1="4.92" x2="3.6272" y2="4.9022" width="0.2032" layer="16"/>
 <wire x1="3.6272" y1="4.9022" x2="3.5306" y2="4.9022" width="0.2032" layer="16"/>
+<contactref element="SH1" pad="FIT@2"/>
+<contactref element="SH1" pad="FIT@1"/>
+<contactref element="SH1" pad="2"/>
+<contactref element="R6" pad="2"/>
+<contactref element="R10" pad="2"/>
+<contactref element="U3" pad="P$15"/>
+<contactref element="U3" pad="A1B12"/>
+<contactref element="U3" pad="B11A12"/>
+<contactref element="U3" pad="P$14"/>
+<contactref element="U3" pad="P$13"/>
+<contactref element="U3" pad="P$16"/>
+<wire x1="88.7845" y1="37.721" x2="89.6995" y2="36.626" width="0" layer="19" extent="16-16"/>
+<wire x1="89.6995" y1="30.176" x2="88.7845" y2="29.081" width="0" layer="19" extent="16-16"/>
+<wire x1="86.214" y1="26.424" x2="84.6045" y2="29.081" width="0" layer="19" extent="16-16"/>
+<wire x1="62.6" y1="33.274" x2="56.515" y2="33.147" width="0" layer="19" extent="16-16"/>
+<wire x1="67.807" y1="37.973" x2="62.6" y2="33.274" width="0" layer="19" extent="16-16"/>
+<wire x1="88.539" y1="17.074" x2="86.214" y2="26.424" width="0" layer="19" extent="16-16"/>
+<wire x1="86.214" y1="14.724" x2="88.539" y2="17.074" width="0" layer="19" extent="16-16"/>
 </signal>
 <signal name="SCL">
@@
 <wire x1="14.854" y1="33.25" x2="14.881" y2="33.223" width="0.3048" layer="16"/>
 <contactref element="U$14" pad="1"/>
+<contactref element="SH1" pad="3"/>
 <wire x1="80.518" y1="82.7024" x2="77.2806" y2="88.1046" width="0" layer="19" extent="1-1"/>
 </signal>
@@
 <wire x1="69.8136" y1="90.667" x2="69.1188" y2="89.9722" width="0.2032" layer="1"/>
 <wire x1="69.1188" y1="89.9722" x2="69.1188" y2="88.3037" width="0.2032" layer="1"/>
-</signal>
-<signal name="N$1">
-<contactref element="U2" pad="B4A9"/>
-<contactref element="U2" pad="A4B9"/>
-<contactref element="IC2" pad="3"/>
-<via x="65.8876" y="86.7664" extent="1-16" drill="0.45"/>
-<wire x1="65.8876" y1="86.7664" x2="70.3072" y2="86.7664" width="0.3048" layer="16"/>
-<via x="70.3072" y="86.7664" extent="1-16" drill="0.45"/>
-<wire x1="70.32" y1="86.7792" x2="70.3072" y2="86.7664" width="0.3048" layer="1"/>
-<wire x1="65.4438" y1="88.3037" x2="65.4438" y2="86.9562" width="0.254" layer="1"/>
-<wire x1="65.8876" y1="86.7664" x2="65.6336" y2="86.7664" width="0.254" layer="1"/>
-<wire x1="65.6336" y1="86.7664" x2="65.4438" y2="86.9562" width="0.254" layer="1"/>
-<wire x1="70.2938" y1="88.3037" x2="70.2938" y2="86.8054" width="0.254" layer="1"/>
-<wire x1="70.2938" y1="86.8054" x2="70.32" y2="86.7792" width="0.254" layer="1"/>
-<contactref element="C29" pad="2"/>
-<wire x1="70.3072" y1="86.7664" x2="71.1598" y2="85.9138" width="0.254" layer="1"/>
-<wire x1="71.1598" y1="85.9138" x2="72.517" y2="85.9138" width="0.254" layer="1"/>
-<wire x1="74.9946" y1="88.1046" x2="72.8038" y2="85.9138" width="0.254" layer="1"/>
-<wire x1="72.8038" y1="85.9138" x2="72.517" y2="85.9138" width="0.254" layer="1"/>
 </signal>
 <signal name="USB_DN">
@@
 <wire x1="64.1604" y1="71.4502" x2="63.3476" y2="72.263" width="0.1524" layer="16"/>
 </signal>
+<signal name="+5V">
+<contactref element="U2" pad="B4A9"/>
+<contactref element="U2" pad="A4B9"/>
+<contactref element="IC2" pad="3"/>
+<contactref element="C29" pad="2"/>
+<via x="65.8876" y="86.7664" extent="1-16" drill="0.45"/>
+<wire x1="65.8876" y1="86.7664" x2="70.3072" y2="86.7664" width="0.3048" layer="16"/>
+<via x="70.3072" y="86.7664" extent="1-16" drill="0.45"/>
+<wire x1="70.32" y1="86.7792" x2="70.3072" y2="86.7664" width="0.3048" layer="1"/>
+<wire x1="65.4438" y1="88.3037" x2="65.4438" y2="86.9562" width="0.254" layer="1"/>
+<wire x1="65.8876" y1="86.7664" x2="65.6336" y2="86.7664" width="0.254" layer="1"/>
+<wire x1="65.6336" y1="86.7664" x2="65.4438" y2="86.9562" width="0.254" layer="1"/>
+<wire x1="70.2938" y1="88.3037" x2="70.2938" y2="86.8054" width="0.254" layer="1"/>
+<wire x1="70.2938" y1="86.8054" x2="70.32" y2="86.7792" width="0.254" layer="1"/>
+<wire x1="70.3072" y1="86.7664" x2="71.1598" y2="85.9138" width="0.254" layer="1"/>
+<wire x1="71.1598" y1="85.9138" x2="72.517" y2="85.9138" width="0.254" layer="1"/>
+<wire x1="74.9946" y1="88.1046" x2="72.8038" y2="85.9138" width="0.254" layer="1"/>
+<wire x1="72.8038" y1="85.9138" x2="72.517" y2="85.9138" width="0.254" layer="1"/>
+<contactref element="SH1" pad="1"/>
+<wire x1="88.539" y1="16.074" x2="72.517" y2="85.9138" width="0" layer="19" extent="1-16"/>
+</signal>
+<signal name="N$1">
+<contactref element="R6" pad="1"/>
+<contactref element="U3" pad="B5"/>
+<wire x1="64.4" y1="33.274" x2="89.6995" y2="35.151" width="0" layer="19" extent="16-16"/>
+</signal>
+<signal name="N$36">
+<contactref element="R10" pad="1"/>
+<contactref element="U3" pad="A5"/>
+<wire x1="69.607" y1="37.973" x2="89.6995" y2="32.151" width="0" layer="19" extent="16-16"/>
+</signal>
 </signals>

Commit message: adding components
Parts:
- moved SH1 8.93 mm to (87.5, 11.7), turned to 270 degrees
- moved U3 6.99 mm to (86.1, 26.4), turned to 270 degrees
Other:
- outline, holes or cut-outs redrawn
Changed lines of the file:
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@@
 <wire x1="4" y1="96" x2="0" y2="92" width="0" layer="20" curve="90"/>
 <polygon width="0.2032" layer="46">
-<vertex x="82.693" y="14.637"/>
-<vertex x="62.468" y="14.637"/>
-<vertex x="62.468" y="16.034"/>
-<vertex x="82.693" y="16.034"/>
+<vertex x="79.693" y="14.637"/>
+<vertex x="65.468" y="14.637"/>
+<vertex x="65.468" y="16.034"/>
+<vertex x="79.693" y="16.034"/>
 </polygon>
 <text x="87.7316" y="56.5404" size="1.27" layer="26" rot="MR0" align="center">DFU</text>
@@
 <element name="SW21" library="duckypad" package="EVQ-Q2" value="SPST_TACT-EVQQ2" x="65" y="7.5" smashed="yes"/>
 <element name="U$14" library="adafruit_changed" package="1X02" value="PINHD1X2" x="88.9" y="66.675" smashed="yes" rot="R270"/>
-<element name="SH1" library="duckypad" package="DUCKYPAD_SM12B-SSR-H-TB" value="SH10P" x="86.614" y="20.574" smashed="yes" rot="MR90"/>
-<element name="U3" library="my_usbc_16p" package="USBC_16P_FOOT" value="USBC_16P" x="85.852" y="33.401" smashed="yes" rot="MR90"/>
+<element name="SH1" library="duckypad" package="DUCKYPAD_SM12B-SSR-H-TB" value="SH10P" x="87.503" y="11.684" smashed="yes" rot="MR270"/>
+<element name="U3" library="my_usbc_16p" package="USBC_16P_FOOT" value="USBC_16P" x="86.106" y="26.416" smashed="yes" rot="MR270"/>
 <element name="R6" library="joyAnalog" package="0805" value="5.1K" x="63.5" y="33.274" smashed="yes" rot="MR0">
 <attribute name="NAME" x="64.262" y="34.0995" size="0.8128" layer="26" rot="MR0"/>
@@
 <contactref element="U3" pad="P$13"/>
 <contactref element="U3" pad="P$16"/>
-<wire x1="88.7845" y1="37.721" x2="89.6995" y2="36.626" width="0" layer="19" extent="16-16"/>
-<wire x1="89.6995" y1="30.176" x2="88.7845" y2="29.081" width="0" layer="19" extent="16-16"/>
-<wire x1="86.214" y1="26.424" x2="84.6045" y2="29.081" width="0" layer="19" extent="16-16"/>
+<wire x1="83.1735" y1="30.736" x2="82.2585" y2="29.641" width="0" layer="19" extent="16-16"/>
+<wire x1="82.2585" y1="23.191" x2="83.1735" y2="22.096" width="0" layer="19" extent="16-16"/>
+<wire x1="87.903" y1="5.834" x2="83.4" y2="5.25" width="0" layer="19" extent="1-16"/>
+<wire x1="87.903" y1="17.534" x2="87.3535" y2="22.096" width="0" layer="19" extent="16-16"/>
+<wire x1="85.578" y1="15.184" x2="87.903" y2="17.534" width="0" layer="19" extent="16-16"/>
 <wire x1="62.6" y1="33.274" x2="56.515" y2="33.147" width="0" layer="19" extent="16-16"/>
 <wire x1="67.807" y1="37.973" x2="62.6" y2="33.274" width="0" layer="19" extent="16-16"/>
-<wire x1="88.539" y1="17.074" x2="86.214" y2="26.424" width="0" layer="19" extent="16-16"/>
-<wire x1="86.214" y1="14.724" x2="88.539" y2="17.074" width="0" layer="19" extent="16-16"/>
 </signal>
 <signal name="SCL">
@@
 <contactref element="SW21" pad="B'"/>
 <contactref element="SW21" pad="B"/>
-<wire x1="61.219" y1="18.039" x2="61.219" y2="9.75" width="0.2032" layer="1"/>
+<wire x1="61.219" y1="14.229" x2="61.219" y2="9.75" width="0.2032" layer="1"/>
 <wire x1="61.219" y1="9.75" x2="61.6" y2="9.75" width="0.2032" layer="1"/>
-<wire x1="73.787" y1="57.2516" x2="73.787" y2="30.607" width="0.2032" layer="1"/>
-<wire x1="73.787" y1="30.607" x2="61.219" y2="18.039" width="0.2032" layer="1"/>
+<wire x1="73.787" y1="57.2516" x2="73.787" y2="26.797" width="0.2032" layer="1"/>
+<wire x1="73.787" y1="26.797" x2="61.219" y2="14.229" width="0.2032" layer="1"/>
 <wire x1="61.6" y1="9.75" x2="68.4" y2="9.75" width="1.016" layer="1"/>
 </signal>
@@
 <contactref element="SW20" pad="B"/>
 <contactref element="SW20" pad="B'"/>
-<wire x1="74.2188" y1="30.5562" x2="84.074" y2="20.701" width="0.2032" layer="1"/>
-<wire x1="84.074" y1="20.701" x2="84.074" y2="10.424" width="0.2032" layer="1"/>
+<wire x1="74.2188" y1="25.2222" x2="84.074" y2="15.367" width="0.2032" layer="1"/>
+<wire x1="84.074" y1="15.367" x2="84.074" y2="10.424" width="0.2032" layer="1"/>
 <wire x1="84.074" y1="10.424" x2="83.4" y2="9.75" width="0.2032" layer="1"/>
-<wire x1="74.2188" y1="57.511" x2="74.2188" y2="30.5562" width="0.2032" layer="1"/>
+<wire x1="74.2188" y1="57.511" x2="74.2188" y2="25.2222" width="0.2032" layer="1"/>
 <wire x1="76.6" y1="9.75" x2="83.4" y2="9.75" width="1.016" layer="1"/>
 </signal>
@@
 <wire x1="72.8038" y1="85.9138" x2="72.517" y2="85.9138" width="0.254" layer="1"/>
 <contactref element="SH1" pad="1"/>
-<wire x1="88.539" y1="16.074" x2="72.517" y2="85.9138" width="0" layer="19" extent="1-16"/>
+<wire x1="85.578" y1="16.184" x2="72.517" y2="85.9138" width="0" layer="19" extent="1-16"/>
 </signal>
 <signal name="N$1">
 <contactref element="R6" pad="1"/>
 <contactref element="U3" pad="B5"/>
-<wire x1="64.4" y1="33.274" x2="89.6995" y2="35.151" width="0" layer="19" extent="16-16"/>
+<wire x1="64.4" y1="33.274" x2="82.2585" y2="24.666" width="0" layer="19" extent="16-16"/>
 </signal>
 <signal name="N$36">
 <contactref element="R10" pad="1"/>
 <contactref element="U3" pad="A5"/>
-<wire x1="69.607" y1="37.973" x2="89.6995" y2="32.151" width="0" layer="19" extent="16-16"/>
+<wire x1="69.607" y1="37.973" x2="82.2585" y2="27.666" width="0" layer="19" extent="16-16"/>
 </signal>
 </signals>

Commit message: v4 draft done
Parts:
- removed TP1, TP2, TP3, TP5: PTR1TP11SQ, testpad:TP11SQ
- removed TP4: PTR1TP09R, testpad:TP09R
- moved R6 25.7 mm to (85.6, 20.2), turned to 180 degrees
- moved R10 14.6 mm to (82.7, 33.7)
- moved R17 0.86 mm to (69.3, 58.4), turned to 90 degrees
- moved R4 0.13 mm to (85.3, 54.1)
Connections:
- new net N$37: IC1.13, SH1.8
- net +3V3: now also SH1.10
- net +5V: now also U3.A4B9, U3.B4A9
- net BUTTON_DEBUG: no longer IC1.13
- net N$13: now also IC1.19, SH1.7; no longer IC1.20, TP2.TP
- net N$16: now also IC1.22, U3.A7, U3.B7; no longer IC1.21, TP3.TP
- net N$2: now also IC1.20, SH1.6; no longer IC1.19, TP1.TP
- net N$30: now also IC1.21, U3.A6, U3.B6; no longer IC1.22, TP4.TP
- net N$35: now also SH1.5; no longer TP5.TP
Routing:
- net +5V: track 13.8 -> 115.0 mm
- net N$37: track 0.00 -> 83.8 mm, vias 0 -> 1
- net N$13: track 3.40 -> 81.1 mm
- net N$2: track 4.28 -> 81.3 mm
- net N$35: track 5.55 -> 81.4 mm
- net N$30: track 1.53 -> 63.6 mm, vias 0 -> 1
- net N$16: track 3.03 -> 65.0 mm
- net GND: track 154.7 -> 182.9 mm, vias 51 -> 52
- net LED_DATA_EN: track 37.3 -> 28.4 mm
- net N$36: track 0.00 -> 8.38 mm
- net N$1: track 0.00 -> 6.90 mm
- net +3V3: track 99.6 -> 104.5 mm, vias 9 -> 8
- net BUTTON_DEBUG: track 45.2 -> 41.1 mm, vias 3 -> 2
- net N$20: track 24.0 -> 25.6 mm
- net OLED_RESET: track 17.3 -> 18.6 mm
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Other:
- board text removed: "PB1"
- board text removed: "PB10"
- board text removed: "PB11"
- board text removed: "PB12"
- board text removed: "PB2"

Commit message: finishing touches
Routing:
- net N$30: track 63.6 -> 64.5 mm
- net N$16: track 65.0 -> 65.9 mm
- net N$35: track 81.4 -> 82.2 mm
- net N$2: track 81.3 -> 82.0 mm
- net N$13: track 81.1 -> 81.7 mm
