File: pcb/duckypad2020_v4.brd (EAGLE design)
At the start: 90 x 96 mm, 93 parts, among them IC1 STM32F072C8T6, IC2 REG1117, IC3 74AHCT1G08DBV, SW1 324_SW324_SWITCH_FOOT_HOLE, SW10 KAILH_SWITCH_SOCKET_KAILH_SWI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, SW11 KAILH_SWITCH_SOCKET_KAILH_SWI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, SW12 KAILH_SWITCH_SOCKET_KAILH_SWI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, SW13 KAILH_SWITCH_SOCKET_KAILH_SWI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, SW14 KAILH_SWITCH_SOCKET_KAILH_SWI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, SW15 KAILH_SWITCH_SOCKET_KAILH_SWI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

Commit message: adjusted signal names
Connections:
- net BUTTON1 renamed MINUS_BUTTON
- net BUTTON2 renamed PLUS_BUTTON
Changed lines of the file:
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@@
 <wire x1="65.2272" y1="73.7616" x2="55.625" y2="83.3638" width="0.2032" layer="16"/>
 </signal>
-<signal name="BUTTON1">
+<signal name="MINUS_BUTTON">
 <contactref element="IC1" pad="11"/>
 <wire x1="66.25" y1="61.5" x2="66.25" y2="60.8008" width="0.2032" layer="1"/>
@@
 <wire x1="61.6" y1="9.75" x2="68.4" y2="9.75" width="1.016" layer="1"/>
 </signal>
-<signal name="BUTTON2">
+<signal name="PLUS_BUTTON">
 <contactref element="IC1" pad="12"/>
 <wire x1="70.8648" y1="60.865" x2="67.385" y2="60.865" width="0.2032" layer="1"/>
