File: pcb/pcb_plate/evo/duckypad2020_v4.brd (EAGLE design)
At the start: 90 x 96 mm, 13 parts, among them U3 USBC_16P

Commit message: updated PCB plate
Parts:
- removed SH1: SH10P, duckypad:DUCKYPAD_SM12B-SSR-H-TB
- removed U3: USBC_16P, my_usbc_16p:USBC_16P_FOOT
Connections:
- removed net +3V3: SH1.10, SH1.3
- removed net +5V: SH1.1, U3.A4B9, U3.B4A9
- removed net GND: SH1.2, SH1.FIT@1, SH1.FIT@2, U3.A1B12, U3.B11A12, U3.P$13, U3.P$14, U3.P$15, U3.P$16
- removed net N$1: U3.B5
- removed net N$13: SH1.7
- removed net N$16: U3.A7, U3.B7
- removed net N$2: SH1.6
- removed net N$30: U3.A6, U3.B6
- removed net N$35: SH1.5
- removed net N$36: U3.A5
- removed net N$37: SH1.8
Other:
- outline, holes or cut-outs redrawn
Changed lines of the file:
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@@
 <setting verticaltext="up"/>
 </settings>
-<grid distance="0.5" unitdist="mm" unit="mm" style="lines" multiple="1" display="yes" altdistance="1" altunitdist="mil" altunit="mil"/>
+<grid distance="0.25" unitdist="mm" unit="mm" style="lines" multiple="1" display="yes" altdistance="1" altunitdist="mil" altunit="mil"/>
 <layers>
 <layer number="1" name="Top" color="4" fill="1" visible="yes" active="yes"/>
@@
 <wire x1="0" y1="92" x2="0" y2="4" width="0" layer="20"/>
 <wire x1="0" y1="4" x2="4" y2="0" width="0" layer="20" curve="90"/>
-<wire x1="90" y1="3.5" x2="90" y2="1" width="0" layer="20"/>
+<wire x1="85" y1="17.75" x2="85" y2="5.75" width="0" layer="20"/>
+<wire x1="85" y1="5.75" x2="86" y2="4.75" width="0" layer="20" curve="90"/>
+<wire x1="86" y1="4.75" x2="89" y2="4.75" width="0" layer="20"/>
+<wire x1="89" y1="4.75" x2="90" y2="3.75" width="0" layer="20" curve="-90"/>
+<wire x1="90" y1="3.75" x2="90" y2="1" width="0" layer="20"/>
 <wire x1="90" y1="1" x2="89" y2="0" width="0" layer="20" curve="-90"/>
 <wire x1="89" y1="0" x2="4" y2="0" width="0" layer="20"/>
 <wire x1="4" y1="96" x2="86" y2="96" width="0" layer="20"/>
 <wire x1="86" y1="96" x2="90" y2="92" width="0" layer="20" curve="-90"/>
-<wire x1="90" y1="92" x2="90" y2="32.5" width="0" layer="20"/>
+<wire x1="90" y1="92" x2="90" y2="32.75" width="0" layer="20"/>
+<wire x1="90" y1="32.75" x2="89" y2="31.75" width="0" layer="20" curve="-90"/>
+<wire x1="89" y1="31.75" x2="82" y2="31.75" width="0" layer="20"/>
+<wire x1="82" y1="31.75" x2="81" y2="30.75" width="0" layer="20" curve="90"/>
+<wire x1="81" y1="30.75" x2="81" y2="22" width="0" layer="20"/>
+<wire x1="81" y1="22" x2="82" y2="21" width="0" layer="20" curve="90"/>
+<wire x1="82" y1="21" x2="89" y2="21" width="0" layer="20"/>
+<wire x1="89" y1="21" x2="90" y2="20" width="0" layer="20" curve="-90"/>
+<wire x1="90" y1="20" x2="90" y2="19.75" width="0" layer="20"/>
+<wire x1="90" y1="19.75" x2="89" y2="18.75" width="0" layer="20" curve="-90"/>
+<wire x1="89" y1="18.75" x2="86" y2="18.75" width="0" layer="20"/>
+<wire x1="86" y1="18.75" x2="85" y2="17.75" width="0" layer="20" curve="90"/>
 <wire x1="4" y1="96" x2="0" y2="92" width="0" layer="20" curve="90"/>
 <text x="86.7316" y="56.5404" size="1.6764" layer="26" rot="MR0" align="center">DFU</text>
 <text x="86.757" y="49.784" size="1.6764" layer="26" rot="MR180" align="center">RST</text>
 <text x="45" y="7" size="4" layer="26" rot="MR0" align="center">duckyPad.com</text>
-<wire x1="90" y1="32.5" x2="89" y2="31.5" width="0" layer="20" curve="-90"/>
-<wire x1="89" y1="31.5" x2="82" y2="31.5" width="0" layer="20"/>
-<wire x1="82" y1="31.5" x2="81" y2="30.5" width="0" layer="20" curve="90"/>
-<wire x1="81" y1="30.5" x2="81" y2="22" width="0" layer="20"/>
-<wire x1="81" y1="22" x2="82" y2="21" width="0" layer="20" curve="90"/>
-<wire x1="82" y1="21" x2="89" y2="21" width="0" layer="20"/>
-<wire x1="89" y1="21" x2="90" y2="20" width="0" layer="20" curve="-90"/>
-<wire x1="90" y1="20" x2="90" y2="19.5" width="0" layer="20"/>
-<wire x1="90" y1="19.5" x2="89" y2="18.5" width="0" layer="20" curve="-90"/>
-<wire x1="89" y1="18.5" x2="86" y2="18.5" width="0" layer="20"/>
-<wire x1="86" y1="18.5" x2="85" y2="17.5" width="0" layer="20" curve="90"/>
-<wire x1="85" y1="17.5" x2="85" y2="5.5" width="0" layer="20"/>
-<wire x1="85" y1="5.5" x2="86" y2="4.5" width="0" layer="20" curve="90"/>
-<wire x1="86" y1="4.5" x2="89" y2="4.5" width="0" layer="20"/>
-<wire x1="89" y1="4.5" x2="90" y2="3.5" width="0" layer="20" curve="-90"/>
 </plain>
 <attributes>
@@
 <element name="U$13" library="3pos_slide_switch_centered" package="M2_SCREW_FOOT" value="M2_SCREW_DEV" x="38.5" y="19.5" smashed="yes"/>
 <element name="U$23" library="3pos_slide_switch_centered" package="M2_SCREW_FOOT" value="M2_SCREW_DEV" x="82" y="58" smashed="yes"/>
-<element name="SH1" library="duckypad" package="DUCKYPAD_SM12B-SSR-H-TB" value="SH10P" x="87.503" y="11.684" smashed="yes" rot="MR270"/>
-<element name="U3" library="my_usbc_16p" package="USBC_16P_FOOT" value="USBC_16P" x="86.106" y="26.416" smashed="yes" rot="MR270"/>
 <element name="U$1" library="3pos_slide_switch_centered" package="M2_SCREW_FOOT" value="M2_SCREW_DEV" x="72.5" y="12" smashed="yes"/>
 </elements>
 <signals>
-<signal name="GND">
-<contactref element="SH1" pad="FIT@2"/>
-<contactref element="SH1" pad="FIT@1"/>
-<contactref element="SH1" pad="2"/>
-<contactref element="U3" pad="P$15"/>
-<contactref element="U3" pad="A1B12"/>
-<contactref element="U3" pad="B11A12"/>
-<contactref element="U3" pad="P$14"/>
-<contactref element="U3" pad="P$13"/>
-<contactref element="U3" pad="P$16"/>
-<wire x1="83.1735" y1="30.736" x2="87.3535" y2="30.736" width="0" layer="19" extent="1-1"/>
-<wire x1="82.2585" y1="29.641" x2="83.1735" y2="30.736" width="0" layer="19" extent="16-16"/>
-<wire x1="82.2585" y1="23.191" x2="82.2585" y2="29.641" width="0" layer="19" extent="16-16"/>
-<wire x1="83.1735" y1="22.096" x2="82.2585" y2="23.191" width="0" layer="19" extent="16-16"/>
-<wire x1="87.3535" y1="22.096" x2="83.1735" y2="22.096" width="0" layer="19" extent="1-1"/>
-<wire x1="87.903" y1="17.534" x2="87.3535" y2="22.096" width="0" layer="19" extent="16-16"/>
-<wire x1="85.578" y1="15.184" x2="87.903" y2="17.534" width="0" layer="19" extent="16-16"/>
-<wire x1="87.903" y1="5.834" x2="85.578" y2="15.184" width="0" layer="19" extent="16-16"/>
-</signal>
-<signal name="+3V3">
-<contactref element="SH1" pad="3"/>
-<contactref element="SH1" pad="10"/>
-<wire x1="85.578" y1="7.184" x2="85.578" y2="14.184" width="0" layer="19" extent="16-16"/>
-</signal>
-<signal name="+5V">
-<contactref element="SH1" pad="1"/>
-<contactref element="U3" pad="B4A9"/>
-<contactref element="U3" pad="A4B9"/>
-<wire x1="82.2585" y1="23.991" x2="82.2585" y2="28.841" width="0" layer="19" extent="16-16"/>
-<wire x1="85.578" y1="16.184" x2="82.2585" y2="23.991" width="0" layer="19" extent="16-16"/>
-</signal>
-<signal name="N$1">
-<contactref element="U3" pad="B5"/>
-</signal>
-<signal name="N$36">
-<contactref element="U3" pad="A5"/>
-</signal>
-<signal name="N$16">
-<contactref element="U3" pad="A7"/>
-<contactref element="U3" pad="B7"/>
-<wire x1="82.2585" y1="27.166" x2="82.2585" y2="26.166" width="0" layer="19" extent="16-16"/>
-</signal>
-<signal name="N$30">
-<contactref element="U3" pad="A6"/>
-<contactref element="U3" pad="B6"/>
-<wire x1="82.2585" y1="25.666" x2="82.2585" y2="26.666" width="0" layer="19" extent="16-16"/>
-</signal>
-<signal name="N$35">
-<contactref element="SH1" pad="5"/>
-</signal>
-<signal name="N$2">
-<contactref element="SH1" pad="6"/>
-</signal>
-<signal name="N$13">
-<contactref element="SH1" pad="7"/>
-</signal>
-<signal name="N$37">
-<contactref element="SH1" pad="8"/>
-</signal>
 </signals>
 <mfgpreviewcolors>

Commit message: updated plate
Parts:
- removed U$12, U$13, U$8, U$9: M2_SCREW_DEV, 3pos_slide_switch_centered:M2_SCREW_FOOT
Other:
- outline, holes or cut-outs redrawn
Changed lines of the file:
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@@
 <setting verticaltext="up"/>
 </settings>
-<grid distance="0.25" unitdist="mm" unit="mm" style="lines" multiple="1" display="yes" altdistance="1" altunitdist="mil" altunit="mil"/>
+<grid distance="0.5" unitdist="mm" unit="mm" style="lines" multiple="1" display="yes" altdistance="1" altunitdist="mil" altunit="mil"/>
 <layers>
 <layer number="1" name="Top" color="4" fill="1" visible="yes" active="yes"/>
@@
 <wire x1="0" y1="92" x2="0" y2="4" width="0" layer="20"/>
 <wire x1="0" y1="4" x2="4" y2="0" width="0" layer="20" curve="90"/>
-<wire x1="85" y1="17.75" x2="85" y2="5.75" width="0" layer="20"/>
+<wire x1="90" y1="92" x2="90" y2="32.25" width="0" layer="20"/>
+<wire x1="90" y1="32.25" x2="89" y2="31.25" width="0" layer="20" curve="-90"/>
+<wire x1="89" y1="31.25" x2="83" y2="31.25" width="0" layer="20"/>
+<wire x1="83" y1="31.25" x2="82" y2="30.25" width="0" layer="20" curve="90"/>
+<wire x1="82" y1="30.25" x2="82" y2="22.5" width="0" layer="20"/>
+<wire x1="82" y1="22.5" x2="83" y2="21.5" width="0" layer="20" curve="90"/>
+<wire x1="83" y1="21.5" x2="89" y2="21.5" width="0" layer="20"/>
+<wire x1="89" y1="21.5" x2="90" y2="20.5" width="0" layer="20" curve="-90"/>
+<wire x1="90" y1="20.5" x2="90" y2="19.5" width="0" layer="20"/>
+<wire x1="90" y1="19.5" x2="89" y2="18.5" width="0" layer="20" curve="-90"/>
+<wire x1="89" y1="18.5" x2="86" y2="18.5" width="0" layer="20"/>
+<wire x1="86" y1="18.5" x2="85" y2="17.5" width="0" layer="20" curve="90"/>
+<wire x1="85" y1="17.5" x2="85" y2="5.75" width="0" layer="20"/>
 <wire x1="85" y1="5.75" x2="86" y2="4.75" width="0" layer="20" curve="90"/>
 <wire x1="86" y1="4.75" x2="89" y2="4.75" width="0" layer="20"/>
@@
 <wire x1="4" y1="96" x2="86" y2="96" width="0" layer="20"/>
 <wire x1="86" y1="96" x2="90" y2="92" width="0" layer="20" curve="-90"/>
-<wire x1="90" y1="92" x2="90" y2="32.75" width="0" layer="20"/>
-<wire x1="90" y1="32.75" x2="89" y2="31.75" width="0" layer="20" curve="-90"/>
-<wire x1="89" y1="31.75" x2="82" y2="31.75" width="0" layer="20"/>
-<wire x1="82" y1="31.75" x2="81" y2="30.75" width="0" layer="20" curve="90"/>
-<wire x1="81" y1="30.75" x2="81" y2="22" width="0" layer="20"/>
-<wire x1="81" y1="22" x2="82" y2="21" width="0" layer="20" curve="90"/>
-<wire x1="82" y1="21" x2="89" y2="21" width="0" layer="20"/>
-<wire x1="89" y1="21" x2="90" y2="20" width="0" layer="20" curve="-90"/>
-<wire x1="90" y1="20" x2="90" y2="19.75" width="0" layer="20"/>
-<wire x1="90" y1="19.75" x2="89" y2="18.75" width="0" layer="20" curve="-90"/>
-<wire x1="89" y1="18.75" x2="86" y2="18.75" width="0" layer="20"/>
-<wire x1="86" y1="18.75" x2="85" y2="17.75" width="0" layer="20" curve="90"/>
 <wire x1="4" y1="96" x2="0" y2="92" width="0" layer="20" curve="90"/>
 <text x="86.7316" y="56.5404" size="1.6764" layer="26" rot="MR0" align="center">DFU</text>
@@
 <elements>
 <element name="U$7" library="3pos_slide_switch_centered" package="M2_SCREW_FOOT" value="M2_SCREW_DEV" x="19.5" y="19.5" smashed="yes"/>
-<element name="U$9" library="3pos_slide_switch_centered" package="M2_SCREW_FOOT" value="M2_SCREW_DEV" x="38.5" y="76.5" smashed="yes"/>
 <element name="U$10" library="3pos_slide_switch_centered" package="M2_SCREW_FOOT" value="M2_SCREW_DEV" x="82" y="93" smashed="yes"/>
 <element name="U$11" library="3pos_slide_switch_centered" package="M2_SCREW_FOOT" value="M2_SCREW_DEV" x="19.5" y="76.5" smashed="yes"/>
 <element name="U$15" library="3pos_slide_switch_centered" package="M2_SCREW_FOOT" value="M2_SCREW_DEV" x="38.5" y="57.5" smashed="yes"/>
 <element name="U$16" library="3pos_slide_switch_centered" package="M2_SCREW_FOOT" value="M2_SCREW_DEV" x="38.5" y="38.5" smashed="yes"/>
-<element name="U$8" library="3pos_slide_switch_centered" package="M2_SCREW_FOOT" value="M2_SCREW_DEV" x="19.5" y="57.5" smashed="yes"/>
-<element name="U$12" library="3pos_slide_switch_centered" package="M2_SCREW_FOOT" value="M2_SCREW_DEV" x="19.5" y="38.5" smashed="yes"/>
-<element name="U$13" library="3pos_slide_switch_centered" package="M2_SCREW_FOOT" value="M2_SCREW_DEV" x="38.5" y="19.5" smashed="yes"/>
 <element name="U$23" library="3pos_slide_switch_centered" package="M2_SCREW_FOOT" value="M2_SCREW_DEV" x="82" y="58" smashed="yes"/>
 <element name="U$1" library="3pos_slide_switch_centered" package="M2_SCREW_FOOT" value="M2_SCREW_DEV" x="72.5" y="12" smashed="yes"/>
