File: pcb/pcb_plate/evo/duckypad2020_v4.sch (EAGLE design)
At the start: 13 parts, among them U3 USBC_16P

Commit message: updated PCB plate
Parts:
- removed SH1: SH10P, duckypad:SH10P
- removed U3: USBC_16P, my_usbc_16p:USBC_16P
Connections:
- removed net +3V3: SH1.10, SH1.3
- removed net +5V: SH1.1, U3.VBUS
- removed net GND: SH1.11, SH1.12, SH1.2, U3.GND
- removed net N$1: U3.CC2
- removed net N$13: SH1.7
- removed net N$16: U3.DN1, U3.DN2
- removed net N$2: SH1.6
- removed net N$30: U3.DP1, U3.DP2
- removed net N$35: SH1.5
- removed net N$36: U3.CC1
- removed net N$37: SH1.8
Changed lines of the file:
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@@
 <part name="U$13" library="3pos_slide_switch_centered" deviceset="M2_SCREW_DEV" device=""/>
 <part name="U$23" library="3pos_slide_switch_centered" deviceset="M2_SCREW_DEV" device=""/>
-<part name="SH1" library="duckypad" deviceset="SH10P" device=""/>
-<part name="+3V39" library="supply1" library_urn="urn:adsk.eagle:library:371" deviceset="+3V3" device=""/>
-<part name="GND64" library="supply1" deviceset="GND" device=""/>
-<part name="GND5" library="supply1" deviceset="GND" device=""/>
-<part name="P+2" library="supply1" library_urn="urn:adsk.eagle:library:371" deviceset="+5V" device=""/>
-<part name="U3" library="my_usbc_16p" deviceset="USBC_16P" device=""/>
-<part name="GND8" library="supply1" deviceset="GND" device=""/>
-<part name="P+3" library="supply1" library_urn="urn:adsk.eagle:library:371" deviceset="+5V" device=""/>
-<part name="+3V31" library="supply1" library_urn="urn:adsk.eagle:library:371" deviceset="+3V3" device=""/>
 <part name="U$1" library="3pos_slide_switch_centered" deviceset="M2_SCREW_DEV" device=""/>
 </parts>
@@
 <instance part="U$13" gate="G$1" x="495.3" y="2.54" smashed="yes"/>
 <instance part="U$23" gate="G$1" x="467.36" y="17.78" smashed="yes"/>
-<instance part="SH1" gate="G$1" x="388.62" y="-256.54" smashed="yes"/>
-<instance part="+3V39" gate="G$1" x="408.94" y="-246.38" smashed="yes" rot="MR0">
-<attribute name="VALUE" x="411.48" y="-251.46" size="1.778" layer="96" rot="MR90"/>
-</instance>
-<instance part="GND64" gate="1" x="381" y="-276.86" smashed="yes" rot="MR0">
-<attribute name="VALUE" x="383.54" y="-279.4" size="1.778" layer="96" rot="MR0"/>
-</instance>
-<instance part="GND5" gate="1" x="373.38" y="-248.92" smashed="yes" rot="MR0">
-<attribute name="VALUE" x="375.92" y="-251.46" size="1.778" layer="96" rot="MR0"/>
-</instance>
-<instance part="P+2" gate="1" x="373.38" y="-238.76" smashed="yes">
-<attribute name="VALUE" x="370.84" y="-243.84" size="1.778" layer="96" rot="R90"/>
-</instance>
-<instance part="U3" gate="G$1" x="408.94" y="-322.58" smashed="yes" rot="MR0"/>
-<instance part="GND8" gate="1" x="370.84" y="-330.2" smashed="yes" rot="MR0">
-<attribute name="VALUE" x="373.38" y="-332.74" size="1.778" layer="96" rot="MR0"/>
-</instance>
-<instance part="P+3" gate="1" x="439.42" y="-297.18" smashed="yes">
-<attribute name="VALUE" x="436.88" y="-302.26" size="1.778" layer="96" rot="R90"/>
-</instance>
-<instance part="+3V31" gate="G$1" x="411.48" y="-264.16" smashed="yes" rot="MR0">
-<attribute name="VALUE" x="414.02" y="-269.24" size="1.778" layer="96" rot="MR90"/>
-</instance>
 <instance part="U$1" gate="G$1" x="505.46" y="-53.34" smashed="yes"/>
 </instances>
@@
 </busses>
 <nets>
-<net name="GND" class="0">
-<segment>
-<pinref part="SH1" gate="G$1" pin="12"/>
-<pinref part="GND64" gate="1" pin="GND"/>
-<wire x1="386.08" y1="-274.32" x2="381" y2="-274.32" width="0.1524" layer="91"/>
-<pinref part="SH1" gate="G$1" pin="11"/>
-<wire x1="386.08" y1="-271.78" x2="381" y2="-271.78" width="0.1524" layer="91"/>
-<wire x1="381" y1="-271.78" x2="381" y2="-274.32" width="0.1524" layer="91"/>
-<junction x="381" y="-274.32"/>
-</segment>
-<segment>
-<pinref part="SH1" gate="G$1" pin="2"/>
-<pinref part="GND5" gate="1" pin="GND"/>
-<wire x1="386.08" y1="-246.38" x2="373.38" y2="-246.38" width="0.1524" layer="91"/>
-</segment>
-<segment>
-<pinref part="GND8" gate="1" pin="GND"/>
-<wire x1="370.84" y1="-322.58" x2="370.84" y2="-327.66" width="0.1524" layer="91"/>
-<wire x1="370.84" y1="-307.34" x2="370.84" y2="-322.58" width="0.1524" layer="91"/>
-<pinref part="U3" gate="G$1" pin="GND"/>
-<wire x1="424.18" y1="-322.58" x2="370.84" y2="-322.58" width="0.1524" layer="91"/>
-<junction x="370.84" y="-322.58"/>
-</segment>
-</net>
-<net name="+3V3" class="0">
-<segment>
-<pinref part="+3V39" gate="G$1" pin="+3V3"/>
-<pinref part="SH1" gate="G$1" pin="3"/>
-<wire x1="408.94" y1="-248.92" x2="386.08" y2="-248.92" width="0.1524" layer="91"/>
-</segment>
-<segment>
-<pinref part="SH1" gate="G$1" pin="10"/>
-<pinref part="+3V31" gate="G$1" pin="+3V3"/>
-<wire x1="386.08" y1="-266.7" x2="411.48" y2="-266.7" width="0.1524" layer="91"/>
-</segment>
-</net>
-<net name="+5V" class="0">
-<segment>
-<pinref part="SH1" gate="G$1" pin="1"/>
-<pinref part="P+2" gate="1" pin="+5V"/>
-<wire x1="386.08" y1="-243.84" x2="373.38" y2="-243.84" width="0.1524" layer="91"/>
-<wire x1="373.38" y1="-243.84" x2="373.38" y2="-241.3" width="0.1524" layer="91"/>
-</segment>
-<segment>
-<pinref part="U3" gate="G$1" pin="VBUS"/>
-<pinref part="P+3" gate="1" pin="+5V"/>
-<wire x1="424.18" y1="-302.26" x2="439.42" y2="-302.26" width="0.1524" layer="91"/>
-<wire x1="439.42" y1="-302.26" x2="439.42" y2="-299.72" width="0.1524" layer="91"/>
-</segment>
-</net>
-<net name="N$1" class="0">
-<segment>
-<wire x1="383.54" y1="-312.42" x2="381" y2="-312.42" width="0.1524" layer="91"/>
-<wire x1="391.16" y1="-309.88" x2="383.54" y2="-309.88" width="0.1524" layer="91"/>
-<wire x1="383.54" y1="-309.88" x2="383.54" y2="-312.42" width="0.1524" layer="91"/>
-<pinref part="U3" gate="G$1" pin="CC2"/>
-</segment>
-</net>
-<net name="N$36" class="0">
-<segment>
-<wire x1="391.16" y1="-307.34" x2="381" y2="-307.34" width="0.1524" layer="91"/>
-<pinref part="U3" gate="G$1" pin="CC1"/>
-</segment>
-</net>
-<net name="N$16" class="0">
-<segment>
-<pinref part="U3" gate="G$1" pin="DN1"/>
-<wire x1="492.76" y1="-314.96" x2="434.34" y2="-314.96" width="0.1524" layer="91"/>
-<pinref part="U3" gate="G$1" pin="DN2"/>
-<wire x1="434.34" y1="-314.96" x2="424.18" y2="-314.96" width="0.1524" layer="91"/>
-<wire x1="424.18" y1="-317.5" x2="434.34" y2="-317.5" width="0.1524" layer="91"/>
-<wire x1="434.34" y1="-317.5" x2="434.34" y2="-314.96" width="0.1524" layer="91"/>
-<junction x="434.34" y="-314.96"/>
-</segment>
-</net>
-<net name="N$30" class="0">
-<segment>
-<pinref part="U3" gate="G$1" pin="DP1"/>
-<wire x1="424.18" y1="-307.34" x2="431.8" y2="-307.34" width="0.1524" layer="91"/>
-<pinref part="U3" gate="G$1" pin="DP2"/>
-<wire x1="431.8" y1="-307.34" x2="500.38" y2="-307.34" width="0.1524" layer="91"/>
-<wire x1="424.18" y1="-309.88" x2="431.8" y2="-309.88" width="0.1524" layer="91"/>
-<wire x1="431.8" y1="-309.88" x2="431.8" y2="-307.34" width="0.1524" layer="91"/>
-<junction x="431.8" y="-307.34"/>
-</segment>
-</net>
-<net name="N$35" class="0">
-<segment>
-<pinref part="SH1" gate="G$1" pin="5"/>
-<wire x1="386.08" y1="-254" x2="487.68" y2="-254" width="0.1524" layer="91"/>
-</segment>
-</net>
-<net name="N$2" class="0">
-<segment>
-<pinref part="SH1" gate="G$1" pin="6"/>
-<wire x1="510.54" y1="-256.54" x2="386.08" y2="-256.54" width="0.1524" layer="91"/>
-</segment>
-</net>
-<net name="N$13" class="0">
-<segment>
-<pinref part="SH1" gate="G$1" pin="7"/>
-<wire x1="515.62" y1="-259.08" x2="386.08" y2="-259.08" width="0.1524" layer="91"/>
-</segment>
-</net>
-<net name="N$37" class="0">
-<segment>
-<pinref part="SH1" gate="G$1" pin="8"/>
-<wire x1="347.98" y1="-261.62" x2="386.08" y2="-261.62" width="0.1524" layer="91"/>
-</segment>
-</net>
 </nets>
 </sheet>
@@
 </schematic>
 </drawing>
-<compatibility>
-<note version="8.2" severity="warning">
-Since Version 8.2, EAGLE supports online libraries. The ids
-of those online libraries will not be understood (or retained)
-with this version.
-</note>
-<note version="8.3" severity="warning">
-Since Version 8.3, EAGLE supports URNs for individual library
-assets (packages, symbols, and devices). The URNs of those assets
-will not be understood (or retained) with this version.
-</note>
-</compatibility>
 </eagle>

Commit message: updated plate
Parts:
- removed U$12, U$13, U$8, U$9: M2_SCREW_DEV, 3pos_slide_switch_centered:M2_SCREW_DEV
Changed lines of the file:
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@@
 <parts>
 <part name="U$7" library="3pos_slide_switch_centered" deviceset="M2_SCREW_DEV" device=""/>
-<part name="U$9" library="3pos_slide_switch_centered" deviceset="M2_SCREW_DEV" device=""/>
 <part name="U$10" library="3pos_slide_switch_centered" deviceset="M2_SCREW_DEV" device=""/>
 <part name="U$11" library="3pos_slide_switch_centered" deviceset="M2_SCREW_DEV" device=""/>
 <part name="U$15" library="3pos_slide_switch_centered" deviceset="M2_SCREW_DEV" device=""/>
 <part name="U$16" library="3pos_slide_switch_centered" deviceset="M2_SCREW_DEV" device=""/>
-<part name="U$8" library="3pos_slide_switch_centered" deviceset="M2_SCREW_DEV" device=""/>
-<part name="U$12" library="3pos_slide_switch_centered" deviceset="M2_SCREW_DEV" device=""/>
-<part name="U$13" library="3pos_slide_switch_centered" deviceset="M2_SCREW_DEV" device=""/>
 <part name="U$23" library="3pos_slide_switch_centered" deviceset="M2_SCREW_DEV" device=""/>
 <part name="U$1" library="3pos_slide_switch_centered" deviceset="M2_SCREW_DEV" device=""/>
@@
 <instances>
 <instance part="U$7" gate="G$1" x="467.36" y="48.26" smashed="yes"/>
-<instance part="U$9" gate="G$1" x="495.3" y="33.02" smashed="yes"/>
 <instance part="U$10" gate="G$1" x="467.36" y="33.02" smashed="yes"/>
 <instance part="U$11" gate="G$1" x="523.24" y="33.02" smashed="yes"/>
 <instance part="U$15" gate="G$1" x="495.3" y="48.26" smashed="yes"/>
 <instance part="U$16" gate="G$1" x="523.24" y="48.26" smashed="yes"/>
-<instance part="U$8" gate="G$1" x="523.24" y="2.54" smashed="yes"/>
-<instance part="U$12" gate="G$1" x="467.36" y="2.54" smashed="yes"/>
-<instance part="U$13" gate="G$1" x="495.3" y="2.54" smashed="yes"/>
 <instance part="U$23" gate="G$1" x="467.36" y="17.78" smashed="yes"/>
 <instance part="U$1" gate="G$1" x="505.46" y="-53.34" smashed="yes"/>
